Commit message: Update create3.urdf

File: Create3_URDF/create3.urdf (robot description, URDF)
Before this commit: robot create3, 29 links, 28 joints
Links:
- link base_link: geometry collision cylinder length=0.06 radius=0.16399999999999998; visual mesh filename=meshes/body_visual.dae
- link bumper: geometry collision mesh filename=meshes/bumper_collision.dae; visual mesh filename=meshes/bumper_visual.dae

Commit message: Add ZMQ client sample

File: Create3_URDF/create3.urdf (robot description, URDF)
Before this commit: robot create3, 29 links, 28 joints
Links:
- link base_link: geometry collision cylinder length=0.06 radius=0.16399999999999998; visual mesh filename=C:/Users/halle/OneDrive/Documents/Hal/2024-vr-dt/digital-tw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
- link bumper: geometry collision mesh filename=C:/Users/halle/OneDrive/Documents/Hal/2024-vr-dt/digital-tw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; visual mesh filename=C:/Users/halle/OneDrive/Documents/Hal/2024-vr-dt/digital-tw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
