Commit message: Reorganize project files

File: Robot_Files/ER_MyArm300/description/myarm_300_pi.urdf (robot description, URDF)
Before this commit: robot firefighter, 8 links, 7 joints
Links:
- link base: geometry collision mesh filename=base.dae; visual mesh filename=base.dae
- link joint1: geometry collision mesh filename=j1.dae; visual mesh filename=j1.dae
- link joint2: geometry collision mesh filename=j2.dae; visual mesh filename=j2.dae
- link joint3: geometry collision mesh filename=j3.dae; visual mesh filename=j3.dae
- link joint4: geometry collision mesh filename=j4.dae; visual mesh filename=j4.dae
- link joint5: geometry collision mesh filename=j5.dae; visual mesh filename=j5.dae
- link joint6: geometry collision mesh filename=j6.dae; visual mesh filename=j6.dae
- link joint7: geometry collision mesh filename=j7.dae; visual mesh filename=j7.dae

Commit message: Add HandTracking Unity Project

File: Robot_Files/ER_MyArm300/description/myarm_300_pi.urdf (robot description, URDF)
Before this commit: robot firefighter, 8 links, 7 joints
Joints:
- joint joint1_to_base: limit lower=-2.7925 upper=2.7925 effort=1000.0 velocity=2 -> lower=-2.7925 upper=2.7925 effort=1000.0 velocity=1
- joint joint2_to_joint1: limit lower=-1.3962 upper=1.3962 effort=1000.0 velocity=2 -> lower=-1.3962 upper=1.3962 effort=1000.0 velocity=1
- joint joint3_to_joint2: limit lower=-2.8797 upper=2.8797 effort=1000.0 velocity=2 -> lower=-2.8797 upper=2.8797 effort=1000.0 velocity=1
- joint joint4_to_joint3: limit lower=-1.7453 upper=1.3962 effort=1000.0 velocity=2 -> lower=-1.7453 upper=1.3962 effort=1000.0 velocity=1
- joint joint5_to_joint4: limit lower=-2.8797 upper=2.8797 effort=1000.0 velocity=2 -> lower=-2.8797 upper=2.8797 effort=1000.0 velocity=1
- joint joint6_to_joint5: limit lower=-1.9198 upper=1.9198 effort=1000.0 velocity=2 -> lower=-1.9198 upper=1.9198 effort=1000.0 velocity=1
- joint joint7_to_joint6: limit lower=-2.8797 upper=2.8797 effort=1000.0 velocity=2 -> lower=-2.8797 upper=2.8797 effort=1000.0 velocity=1
